File: hardware/hl2_6xvtr.kicad_pcb (KiCad board)
At the start: 2 copper layers, 100 x 49.9 mm, 127 parts, among them J1 Conn_Coaxial-Connector, J10 RCJ-041, J2 Conn_Coaxial-Connector, J3 Conn_Coaxial-Connector, J4 Conn_Coaxial-Connector, J5 Conn_Coaxial-Connector, J6 Conn_01x20, P1 CONN_01X03, Q5 BC807, Q6 SI2309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

Commit message: R2 schem, PCB and gerbers
Fixes #1, fixes #4, fixes #5
Parts:
- removed G***: OSHW-logo_silkscreen-front_2mm, N2ADR:OSHW-logo_silkscreen-front_2mm
- removed R5, R7: DNF, hermeslite:SMD-0603_r
- removed R6: 0R, hermeslite:SMD-0603_r
- removed REF** (x20): via, Local:via30
- added C49: 1u, hermeslite:SMD-0603_c, F.Cu at (126.4, 69.0)
- added C50: 1n, hermeslite:SMD-0603_c, B.Cu at (122.7, 69.5)
- added C51: 1u, hermeslite:SMD-0603_c, F.Cu at (154.8, 81.2)
- added L7: 470nH, hermeslite:SMD-0805, B.Cu at (146.4, 82.8)
- added U7: PGA-105, n2adr:SOT-89-3_round, F.Cu at (123.7, 72.3)
- C21, C30: value 8.6p -> 10p
- C24, C28: value 1p -> 1.8p
- C38, C45: value 9.5p -> 10p
- C41, C48: value 13.7p -> 15p
- C43: value 1.7p -> 1.8p
- R1, R3: value DNF -> 150R; footprint hermeslite:SMD-0603_r -> hermeslite:SMD-0805
- R2: value 0R -> 38R; footprint hermeslite:SMD-0603_r -> hermeslite:SMD-0805
- U1, U3, U4: footprint Package_TO_SOT_SMD:SOT-89-3 -> n2adr:SOT-89-3_round
- U5: value SPF5189Z -> 74LVC1G04; footprint Package_TO_SOT_SMD:SOT-89-3 -> Package_TO_SOT_SMD:SOT-353_SC-70-5_Handsoldering
- moved R1 11.6 mm to (119.4, 72.7)
- moved R2 11.2 mm to (117.5, 76.2)
- moved R3 10.7 mm to (115.4, 72.8)
- moved U5 6.77 mm to (125.7, 66.8), turned to 180 degrees
- moved C6 2.30 mm to (129.4, 72.1)
- moved C19 2.14 mm to (129.4, 74.2)
- moved C12 2.03 mm to (121.3, 76.1)
- moved L1 2.03 mm to (127.7, 76.1)
- moved C4 1.60 mm to (122.0, 66.9), turned to 90 degrees
- moved J1 1.41 mm to (130.8, 66.8)
- moved U2 0.41 mm to (110.7, 78.7)
- moved C25 0.33 mm to (144.4, 58.4)
Connections:
- C8 pad 1: Net-(C8-Pad1) -> HL2TX
- D2 pad 1: INTTR -> EXTTR
- J10 pad 2: INTTR -> EXTTR
- R1 pad 1: /HL2_CLK -> Net-(C12-Pad2)
- R2 pad 1: Net-(C4-Pad2) -> Net-(R2-Pad1)
- R2 pad 2: /HL2_CLK -> Net-(C12-Pad2)
- R3 pad 1: Net-(C4-Pad2) -> Net-(R2-Pad1)
- U2 pad 6: Net-(C12-Pad2) -> Net-(R2-Pad1)
- U5 pad 1: Net-(C4-Pad1) -> (no net)
- U5 pad 2: GND -> /HL2_CLK
- U5 pad 3: Net-(C12-Pad1) -> GND
Routing:
- net EXTTR: track 0.00 -> 87.9 mm, vias 0 -> 1
- net INTTR: track 80.6 -> 0.00 mm, vias 1 -> 0
- net +3V3: track 0.00 -> 50.1 mm, vias 0 -> 3
- net +5VTX: track 100.1 -> 110.2 mm
- net HL2TX: track 6.61 -> 12.7 mm
- net Net-(R2-Pad1): track 0.00 -> 5.85 mm
- net /HL2_CLK: track 7.00 -> 2.70 mm
- net Net-(C8-Pad1): track 4.04 -> 0.00 mm
- net GND: track 140.4 -> 144.1 mm, vias 0 -> 93
- net Net-(C30-Pad2): track 3.27 -> 5.97 mm
- net Net-(C4-Pad2): track 4.95 -> 2.36 mm
- net +5V: track 80.2 -> 77.8 mm
- net +5VRX: track 119.5 -> 117.4 mm
- net Net-(C25-Pad1): track 12.2 -> 13.9 mm
