File: hardware/hl2_6xvtr.sch (KiCad schematic (older format))
At the start: 106 parts, among them J1 Conn_Coaxial-Connector, J10 RCJ-041, J2 Conn_Coaxial-Connector, J3 Conn_Coaxial-Connector, J4 Conn_Coaxial-Connector, J5 Conn_Coaxial-Connector, J6 Conn_01x20, P1 CONN_01X03, Q5 BC807, Q6 SI2309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

Commit message: Fixes #6, #2, partial #1, #4
Parts:
- removed R5, R7: DNF, hermeslite:SMD-0603_r, symbol hl2_6xvtr:R
- removed R6: 0R, hermeslite:SMD-0603_r, symbol hl2_6xvtr:R
- removed U5: SPF5189Z, Package_TO_SOT_SMD:SOT-89-3, symbol hl2_6xvtr:SPF5189Z
- added C? (x2): 1u, hermeslite:SMD-0603_c, symbol hl2_6xvtr:C_Small
- added C?: 1n, hermeslite:SMD-0603_c, symbol hl2_6xvtr:C_Small
- added L?: 470nH, hermeslite:SMD-0805, symbol hl2_6xvtr:L_Small-Device
- added U?: PGA-105, Package_TO_SOT_SMD:SOT-89-3, symbol hl2_6xvtr:PGA-105
- added U?: 74LVC1G04, Package_TO_SOT_SMD:SOT-353_SC-70-5_Handsoldering, symbol 74xGxx:74LVC1G04
- C21, C30: value 8.6p -> 10p
- C24, C28: value 1p -> 1.8p
- C38, C45: value 9.5p -> 10p
- C41, C48: value 13.7p -> 15p
- C43: value 1.7p -> 1.8p
- R1, R2, R3: footprint hermeslite:SMD-0603_r -> hermeslite:SMD-0805
Connections:
- net +3V3: now also C?.2, C?.2, U?.5 (VCC)
- net +5VTX: now also C?.2
- net EXTTR: now also D2.1 (K), J10.2
- net GND: now also C?.1, C?.1, C?.1, L?.2, U?.2 (GND), U?.3 (GND)
- net HL2TX: now also C8.1
- net HL2_CLK: now also U?.2; no longer R1.1, R2.2
- net INTTR: no longer D2.1 (K), J10.2
- net at R2.1, R3.1: now also U2.6 (LO); no longer C4.2
- net at C12.2: now also R1.1, R2.2; no longer U2.6 (LO)
- net at C30.2, D1.3 (K): now also L?.1
- net at C4.1: now also U?.1
- net at C12.1, L1.2: now also U?.3
- new net: C4.2, U?.4
Other:
- note added: "To reduce heat, instead of 12 V from HL2, use Vpa on HL2 board (8 V)"
- moved on the sheet: C12, C19, C21, C23, C24, C26, C27, C28, C29, C30, C32, C33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

Commit message: R2 schem, PCB and gerbers
Fixes #1, fixes #4, fixes #5
Parts:
- R1, R3: value DNF -> 150R
- R2: value 0R -> 38R
- U1, U3, U4: footprint Package_TO_SOT_SMD:SOT-89-3 -> n2adr:SOT-89-3_round
- U7: renamed from U?; footprint Package_TO_SOT_SMD:SOT-89-3 -> n2adr:SOT-89-3_round
- gave numbers to parts that had none: 5
Other:
- note added: "6 dB attenuator"
Changed lines of the file:
@@
 F 0 "U3" H 11700 8542 50  0000 C CNN
 F 1 "SPF5189Z" H 11700 8451 50  0000 C CNN
-F 2 "Package_TO_SOT_SMD:SOT-89-3" H 11750 8575 50  0001 C CNN
+F 2 "n2adr:SOT-89-3_round" H 11750 8575 50  0001 C CNN
 F 3 "www.qorvo.com/products/d/da001910" H 11700 8175 50  0001 C CNN
 F 4 "Mouser: 772-SPF5189Z" H 11700 8175 50  0001 C CNN "Vendor"
@@
 F 0 "U4" H 12000 6742 50  0000 C CNN
 F 1 "SPF5189Z" H 12000 6651 50  0000 C CNN
-F 2 "Package_TO_SOT_SMD:SOT-89-3" H 12050 6775 50  0001 C CNN
+F 2 "n2adr:SOT-89-3_round" H 12050 6775 50  0001 C CNN
 F 3 "www.qorvo.com/products/d/da001910" H 12000 6375 50  0001 C CNN
 F 4 "Mouser: 772-SPF5189Z" H 12000 6375 50  0001 C CNN "Vendor"
@@
 F 0 "U1" H 4250 6817 50  0000 C CNN
 F 1 "PGA-105" H 4250 6726 50  0000 C CNN
-F 2 "Package_TO_SOT_SMD:SOT-89-3" H 4300 6850 50  0001 C CNN
+F 2 "n2adr:SOT-89-3_round" H 4300 6850 50  0001 C CNN
 F 3 "https://www.minicircuits.com/pdfs/PGA-105+.pdf" H 4250 6450 50  0001 C CNN
 F 4 "Mouser: 139-PGA-105" H 4250 6450 50  0001 C CNN "Vendor"
@@
 P 6075 10675
 F 0 "R3" H 6145 10721 50  0000 L CNN
-F 1 "DNF" H 6145 10630 50  0000 L CNN
+F 1 "150R" H 6145 10630 50  0000 L CNN
 F 2 "hermeslite:SMD-0805" V 6005 10675 50  0001 C CNN
 F 3 "" H 6075 10675 50  0001 C CNN
@@
 U 1 1 60541A32
 P 5800 10350
-F 0 "R2" H 5870 10396 50  0000 L CNN
-F 1 "0R" H 5870 10305 50  0000 L CNN
+F 0 "R2" V 5900 10150 50  0000 L CNN
+F 1 "38R" V 5900 10375 50  0000 L CNN
 F 2 "hermeslite:SMD-0805" V 5730 10350 50  0001 C CNN
 F 3 "" H 5800 10350 50  0001 C CNN
@@
 P 5525 10675
 F 0 "R1" H 5595 10721 50  0000 L CNN
-F 1 "DNF" H 5595 10630 50  0000 L CNN
+F 1 "150R" H 5595 10630 50  0000 L CNN
 F 2 "hermeslite:SMD-0805" V 5455 10675 50  0001 C CNN
 F 3 "" H 5525 10675 50  0001 C CNN
@@
 	13525 1425 13525 1700
 $Comp
-L hl2_6xvtr:PGA-105 U?
+L hl2_6xvtr:PGA-105 U7
 U 1 1 613AFF4B
 P 3975 10350
-F 0 "U?" H 3975 10717 50  0000 C CNN
+F 0 "U7" H 3975 10717 50  0000 C CNN
 F 1 "PGA-105" H 3975 10626 50  0000 C CNN
-F 2 "Package_TO_SOT_SMD:SOT-89-3" H 4025 10750 50  0001 C CNN
+F 2 "n2adr:SOT-89-3_round" H 4025 10750 50  0001 C CNN
 F 3 "https://www.minicircuits.com/pdfs/PGA-105+.pdf" H 3975 10350 50  0001 C CNN
 F 4 "Mouser: 139-PGA-105" H 3975 10350 50  0001 C CNN "Vendor"
@@
 Connection ~ 5525 10350
 $Comp
-L hl2_6xvtr:C_Small C?
+L hl2_6xvtr:C_Small C51
 U 1 1 614B2BF9
 P 10400 5750
-F 0 "C?" H 10625 5700 50  0000 C CNN
+F 0 "C51" H 10625 5700 50  0000 C CNN
 F 1 "1u" H 10575 5775 50  0000 C CNN
 F 2 "hermeslite:SMD-0603_c" H 10400 5750 50  0001 C CNN
@@
 $EndComp
 $Comp
-L hl2_6xvtr:GND #PWR?
+L hl2_6xvtr:GND #PWR012
 U 1 1 614B3C0E
 P 10400 5875
-F 0 "#PWR?" H 10400 5625 50  0001 C CNN
+F 0 "#PWR012" H 10400 5625 50  0001 C CNN
 F 1 "GND" H 10405 5702 50  0000 C CNN
 F 2 "" H 10400 5875 50  0001 C CNN
@@
 Connection ~ 10850 5525
 $Comp
-L hl2_6xvtr:L_Small-Device L?
+L hl2_6xvtr:L_Small-Device L7
 U 1 1 614E4B34
 P 10150 7575
-F 0 "L?" H 10198 7621 50  0000 L CNN
+F 0 "L7" H 10198 7621 50  0000 L CNN
 F 1 "470nH" H 10198 7530 50  0000 L CNN
 F 2 "hermeslite:SMD-0805" H 10150 7575 50  0001 C CNN
@@
 	10150 7300 10750 7300
 $Comp
-L hl2_6xvtr:GND #PWR?
+L hl2_6xvtr:GND #PWR011
 U 1 1 615AA36F
 P 10150 7800
-F 0 "#PWR?" H 10150 7550 50  0001 C CNN
+F 0 "#PWR011" H 10150 7550 50  0001 C CNN
 F 1 "GND" H 10155 7627 50  0000 C CNN
 F 2 "" H 10150 7800 50  0001 C CNN
@@
 	10150 7675 10150 7800
 $Comp
-L 74xGxx:74LVC1G04 U?
+L 74xGxx:74LVC1G04 U5
 U 1 1 616BA199
 P 2525 10350
-F 0 "U?" H 2500 10617 50  0000 C CNN
-F 1 "74LVC1G04" H 2500 10526 50  0000 C CNN
+F 0 "U5" H 2625 10600 50  0000 C CNN
+F 1 "74LVC1G04" H 2775 10500 50  0000 C CNN
 F 2 "Package_TO_SOT_SMD:SOT-353_SC-70-5_Handsoldering" H 2525 10350 50  0001 C CNN
 F 3 "http://www.ti.com/lit/sg/scyt129e/scyt129e.pdf" H 2525 10350 50  0001 C CNN
@@
 $EndComp
 $Comp
-L hl2_6xvtr:GND #PWR?
+L hl2_6xvtr:GND #PWR08
 U 1 1 616FB53B
 P 2300 9825
-F 0 "#PWR?" H 2300 9575 50  0001 C CNN
+F 0 "#PWR08" H 2300 9575 50  0001 C CNN
 F 1 "GND" H 2305 9652 50  0000 C CNN
 F 2 "" H 2300 9825 50  0001 C CNN
@@
 	2300 9825 2300 9800
 $Comp
-L hl2_6xvtr:C_Small C?
+L hl2_6xvtr:C_Small C50
 U 1 1 616FB934
 P 2300 9700
-F 0 "C?" H 2525 9650 50  0000 C CNN
+F 0 "C50" H 2525 9650 50  0000 C CNN
 F 1 "1n" H 2475 9725 50  0000 C CNN
 F 2 "hermeslite:SMD-0603_c" H 2300 9700 50  0001 C CNN
@@
 $EndComp
 $Comp
-L hl2_6xvtr:C_Small C?
+L hl2_6xvtr:C_Small C49
 U 1 1 616FB93E
 P 1925 9700
-F 0 "C?" H 2150 9650 50  0000 C CNN
+F 0 "C49" H 2150 9650 50  0000 C CNN
 F 1 "1u" H 2100 9725 50  0000 C CNN
 F 2 "hermeslite:SMD-0603_c" H 1925 9700 50  0001 C CNN
@@
 $EndComp
 $Comp
-L hl2_6xvtr:GND #PWR?
+L hl2_6xvtr:GND #PWR07
 U 1 1 616FB948
 P 1925 9825
-F 0 "#PWR?" H 1925 9575 50  0001 C CNN
+F 0 "#PWR07" H 1925 9575 50  0001 C CNN
 F 1 "GND" H 1930 9652 50  0000 C CNN
 F 2 "" H 1925 9825 50  0001 C CNN
@@
 Connection ~ 2300 9475
 $Comp
-L hl2_6xvtr:+3.3V #PWR?
+L hl2_6xvtr:+3.3V #PWR09
 U 1 1 617280A7
 P 2525 9400
-F 0 "#PWR?" H 2525 9250 50  0001 C CNN
+F 0 "#PWR09" H 2525 9250 50  0001 C CNN
 F 1 "+3.3V" H 2540 9573 50  0000 C CNN
 F 2 "" H 2525 9400 50  0001 C CNN
@@
 	1100 10350 2225 10350
 $Comp
-L hl2_6xvtr:GND #PWR?
+L hl2_6xvtr:GND #PWR010
 U 1 1 6178FC79
 P 2525 10700
-F 0 "#PWR?" H 2525 10450 50  0001 C CNN
+F 0 "#PWR010" H 2525 10450 50  0001 C CNN
 F 1 "GND" H 2530 10527 50  0000 C CNN
 F 2 "" H 2525 10700 50  0001 C CNN
@@
 Wire Wire Line
 	1000 7875 3225 7875
+Text Notes 5525 10225 0    50   ~ 0
+6 dB attenuator
 $EndSCHEMATC

Commit message: Add 2m component values to schematic and BoM
Parts:
- C39: value 62p -> 56p
- R38: value 220k -> 150k
Other:
- note added: "0.5p"
- note added: "1) 50 MHz - Triple-tuned band pass filter (see EMRFD), \n Approx 3 MHz BW, 4 dB IL (green)\n2) 144 MHz (blue)"
- note added: "1) 50.3 MHz BPF, 1.6 dB IL BW 5 MHz (green)"
- note added: "1.2p"
- note added: "10p"
- note added: "150 nH"
- note added: "2) 1.2 dB IL, 20 MHz bw 144.5 MHz (BLUE)"
- note added: "2.7p"
- note added: "2.7p\n4.7p"
- note added: "220nH"
- note added: "3.3p"
- note added: "33p"
- note added: "4.7p"
- note added: "5.6p"
- note added: "68n"
- note added: "8.2p"
- note removed: "50.3 MHz BPF\n1.6 dB IL BW 5 MHz"
- note removed: "Triple-tuned band pass filter (see EMRFD)\nApprox 3 MHz BW, 4 dB IL"
Changed lines of the file:
@@
 Connection ~ 11300 8175
 Text Notes 12750 7650 0    50   ~ 0
-50.3 MHz BPF\n1.6 dB IL BW 5 MHz
+1) 50.3 MHz BPF, 1.6 dB IL BW 5 MHz (green)
 Wire Wire Line
 	10850 8525 10850 8575
@@
 Wire Wire Line
 	10850 5525 11200 5525
-Text Notes 7775 6950 0    50   ~ 0
-Triple-tuned band pass filter (see EMRFD)\nApprox 3 MHz BW, 4 dB IL
+Text Notes 7600 6825 0    50   ~ 0
+1) 50 MHz - Triple-tuned band pass filter (see EMRFD), \n    Approx 3 MHz BW, 4 dB IL (green)\n2) 144 MHz (blue)
 Wire Wire Line
 	14075 8175 14350 8175
@@
 P 12525 6625
 F 0 "C39" H 12433 6579 50  0000 R CNN
-F 1 "62p" H 12433 6670 50  0000 R CNN
+F 1 "56p" H 12433 6670 50  0000 R CNN
 F 2 "hermeslite:SMD-0603_c" H 12525 6625 50  0001 C CNN
 F 3 "" H 12525 6625 50  0001 C CNN
@@
 U 1 1 61D7B977
 P 12525 5725
-F 0 "L16" H 12573 5771 50  0000 L CNN
-F 1 "470nH" H 12573 5680 50  0000 L CNN
+F 0 "L16" H 12350 5825 50  0000 L CNN
+F 1 "470nH" H 12250 5750 50  0000 L CNN
 F 2 "hermeslite:SMD-0805" H 12525 5725 50  0001 C CNN
 F 3 "" H 12525 5725 50  0001 C CNN
@@
 P 4325 3600
 F 0 "R38" V 4225 3550 50  0000 L CNN
-F 1 "220k" V 4150 3550 50  0000 L CNN
+F 1 "150k" V 4150 3550 50  0000 L CNN
 F 2 "hermeslite:SMD-0603_r" V 4255 3600 50  0001 C CNN
 F 3 "" H 4325 3600 50  0001 C CNN
@@
 Text Notes 5525 10225 0    50   ~ 0
 6 dB attenuator
+Text Notes 12100 7875 0    50   ~ 0
+2.7p
+Text Notes 13875 7875 0    50   ~ 0
+2.7p
+Text Notes 13475 8325 0    50   ~ 0
+5.6p
+Text Notes 12625 8325 0    50   ~ 0
+5.6p
+Text Notes 13075 7900 0    50   ~ 0
+0.5p
+Text Notes 13775 8550 0    50   ~ 0
+150 nH
+Text Notes 12625 6800 0    50   ~ 0
+10p
+Text Notes 13325 6825 0    50   ~ 0
+33p
+Text Notes 14025 6825 0    50   ~ 0
+8.2p
+Text Notes 13575 6550 0    50   ~ 0
+3.3p
+Text Notes 12850 6525 0    50   ~ 0
+1.2p
+Text Notes 12825 5750 0    50   ~ 0
+68n
+Text Notes 13550 5750 0    50   ~ 0
+68n
+Text Notes 12750 7750 0    50   ~ 0
+2) 1.2 dB IL, 20 MHz bw 144.5 MHz (BLUE)
+Text Notes 8000 7425 0    50   ~ 0
+0.5p
+Text Notes 9100 7425 0    50   ~ 0
+0.5p
+Text Notes 8375 7475 0    50   ~ 0
+2.7p\n4.7p
+Text Notes 7200 7000 0    50   ~ 0
+3.3p
+Text Notes 9800 6975 0    50   ~ 0
+3.3p
+Text Notes 9375 7450 0    50   ~ 0
+4.7p
+Text Notes 7600 7475 0    50   ~ 0
+4.7p
+Text Notes 9575 8175 0    50   ~ 0
+220nH
+Text Notes 7800 8200 0    50   ~ 0
+220nH
+Wire Notes Line
+	10075 8275 10075 6500
+Wire Notes Line
+	12600 5350 12600 6125
+Wire Notes Line
+	12600 6125 12375 6125
+Wire Notes Line
+	12375 6125 12375 7075
+Wire Notes Line
+	12375 7075 15175 7075
+Wire Notes Line
+	15175 7075 15175 5350
+Wire Notes Line
+	15175 5350 12600 5350
+Wire Notes Line
+	12000 7375 12000 9425
+Wire Notes Line
+	12000 9425 14775 9425
+Wire Notes Line
+	14775 9425 14775 7375
+Wire Notes Line
+	14775 7375 12000 7375
+Wire Notes Line
+	7050 6500 7050 8275
+Text Notes 12900 8575 0    50   ~ 0
+150 nH
+Text Notes 9675 7725 0    50   ~ 0
+150 nH
+Text Notes 8975 7725 0    50   ~ 0
+150 nH
+Text Notes 7925 7775 0    50   ~ 0
+150 nH
+Wire Notes Line
+	7050 6500 10075 6500
+Wire Notes Line
+	10075 8275 7050 8275
 $EndSCHEMATC
